Commit message: fix: fix configs

File: assets/BD.urdf (robot description, URDF)
Before this commit: robot BD, 11 links, 10 joints
Links:
- link L4_Link_ankle: geometry collision box size=0.090 0.050 0.018; visual mesh filename=./meshes/L4_Link_ankle.STL
- link R4_Link_ankle: geometry collision box size=0.090 0.050 0.018; visual mesh filename=./meshes/R4_Link_ankle.STL
