Commit message: feat: add dynamic height and target length in play.py

File: assets/BD_old.urdf (robot description, URDF)
Before this commit: robot BD, 11 links, 10 joints
Links:
- link L0_Link: geometry collision cylinder length=0.050 radius=0.025; visual mesh filename=./meshes/L0_Link.STL
- link L1_Link: geometry collision sphere radius=0.015; visual mesh filename=./meshes/L1_Link.STL
- link L2_Link: geometry collision cylinder length=0.130 radius=0.028; visual mesh filename=./meshes/L2_Link.STL
- link L4_Link_ankle: geometry collision box size=0.090 0.050 0.018; visual mesh filename=./meshes/L4_Link_ankle.STL
- link R0_Link: geometry collision cylinder length=0.050 radius=0.025; visual mesh filename=./meshes/R0_Link.STL
- link R1_Link: geometry collision sphere radius=0.015; visual mesh filename=./meshes/R1_Link.STL
- link R2_Link: geometry collision cylinder length=0.130 radius=0.028; visual mesh filename=./meshes/R2_Link.STL
- link R4_Link_ankle: geometry collision box size=0.090 0.050 0.018; visual mesh filename=./meshes/R4_Link_ankle.STL
- link base_link: geometry collision box size=0.12 0.20 0.09; visual mesh filename=./meshes/base_link.STL
